File: Hardware/Control/Control.kicad_pcb (KiCad board)
At the start: 4 copper layers, 184.2 x 76.2 mm, 45 parts, among them SW1 EN11-HSM1AF15, SW2 KO128B2007, SW3 Conn_01x06, U1 AVR128DB64x-xPT, U2 ESDALD05UD4, U3 FT230XS-U

Commit message: New control board
Parts:
- moved C16 2.79 mm to (105.5, 107.2)
- moved R10 2.79 mm to (105.5, 102.7)
- moved R14 2.79 mm to (105.5, 109.2)
- moved R8 2.79 mm to (105.5, 96.0)
- moved R9 2.79 mm to (105.5, 99.3)
- moved SW3 2.79 mm to (101.5, 96.6)
Routing:
- net LED_FIRE_B: track 106.2 -> 103.4 mm
- net LED_FIRE_R: track 97.7 -> 95.1 mm
- net LED_FIRE_G: track 104.0 -> 101.7 mm
- net FIRE: track 89.5 -> 88.3 mm
Other:
- board text added: "Laser Control Board Version 2.1 Brian Pepin 2025"
- board text removed: "Laser Control Board Version 2.0 Brian Pepin 2024"
