File: Hardware/Control/Control.kicad_pcb (KiCad board)
At the start: 4 copper layers, 184.2 x 76.2 mm, 45 parts, among them SW1 EN11-HSM1AF15, SW2 KO128B2007, SW3 Conn_01x06, U1 AVR128DB64x-xPT, U2 ESDALD05UD4, U3 FT230XS-U

Commit message: Minor tweaks
Connections:
- net Net-(U2-IO3) renamed /D+
- net Net-(U2-IO4) renamed /D-
- net Net-(U2-VDD) renamed /VBUS
Changed lines of the file:
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@@
 	(net 78 "unconnected-(ISP1-Pin_5-Pad5)")
 	(net 79 "Net-(U3-~{RESET})")
-	(net 80 "Net-(U2-IO3)")
-	(net 81 "Net-(U2-IO4)")
+	(net 80 "/D+")
+	(net 81 "/D-")
 	(net 82 "LED_FIRE_R")
 	(net 83 "LED_FIRE_G")
@@
 	(net 112 "unconnected-(U1-PG4-Pad58)")
 	(net 113 "unconnected-(U1-PG7-Pad61)")
-	(net 114 "Net-(U2-VDD)")
+	(net 114 "/VBUS")
 	(net 115 "unconnected-(U2-IO1-Pad1)")
 	(net 116 "unconnected-(U2-IO2-Pad3)")
@@
 			(remove_unused_layers no)
 			(roundrect_rratio 0.25)
-			(net 114 "Net-(U2-VDD)")
+			(net 114 "/VBUS")
 			(pinfunction "VBUS")
 			(pintype "power_in")
@@
 			(remove_unused_layers no)
 			(roundrect_rratio 0.25)
-			(net 81 "Net-(U2-IO4)")
+			(net 81 "/D-")
 			(pinfunction "D-")
 			(pintype "bidirectional")
@@
 			(remove_unused_layers no)
 			(roundrect_rratio 0.25)
-			(net 80 "Net-(U2-IO3)")
+			(net 80 "/D+")
 			(pinfunction "D+")
 			(pintype "bidirectional")
@@
 			(layers "F.Cu" "F.Paste" "F.Mask")
 			(roundrect_rratio 0.243902)
-			(net 80 "Net-(U2-IO3)")
+			(net 80 "/D+")
 			(pintype "passive")
 		)
@@
 			(layers "F.Cu" "F.Paste" "F.Mask")
 			(roundrect_rratio 0.25)
-			(net 80 "Net-(U2-IO3)")
+			(net 80 "/D+")
 			(pinfunction "IO3")
 			(pintype "bidirectional")
@@
 			(layers "F.Cu" "F.Paste" "F.Mask")
 			(roundrect_rratio 0.25)
-			(net 114 "Net-(U2-VDD)")
+			(net 114 "/VBUS")
 			(pinfunction "VDD")
 			(pintype "power_in")
@@
 			(layers "F.Cu" "F.Paste" "F.Mask")
 			(roundrect_rratio 0.25)
-			(net 81 "Net-(U2-IO4)")
+			(net 81 "/D-")
 			(pinfunction "IO4")
 			(pintype "bidirectional")
@@
 			(layers "F.Cu" "F.Paste" "F.Mask")
 			(roundrect_rratio 0.243902)
-			(net 81 "Net-(U2-IO4)")
-			(pintype "passive")
-		)
+			(net 81 "/D-")
+			(pintype "passive")
+		)
