File: Hardware/TEC/PowerSupply.kicad_sch (KiCad schematic)
At the start: 8 parts, among them Q10 Si7141DP, Q11 Si7141DP, Q9 2N7002PW, U8 TPS7A26

Commit message: Update to kicad 8
Parts:
- Q9: footprint Package_TO_SOT_SMD:SOT-323_SC-70 -> Package_TO_SOT_SMD:SOT-23
