File: Hardware/TEC/TEC.kicad_sch (KiCad schematic)
At the start: 30 parts, among them J1 DEANS, J2 Data, Q1 2N7002PW, Q2 2N7002PW, U1 LP3985-3.0, U2 DAC108S085CISQ, U3 ADC104S021

Commit message: Update to kicad 8
Parts:
- H1, H2, H3, H4: now left out of the parts list
- Q1, Q2: footprint Package_TO_SOT_SMD:SOT-323_SC-70 -> Package_TO_SOT_SMD:SOT-23
