File: Hardware/Power/PowerSupply.kicad_pcb (KiCad board)
At the start: 4 copper layers, 172 x 85 mm, 203 parts, among them Q1 PSMN1R5-25MLHX, Q10 BSS84, Q11 2N7002PW, Q12 2N7002PW, Q13 2N7002PW, Q14 Si7141DP, Q15 BSS84, Q16 Si7141DP, Q17 Si7141DP, Q18 Si7141DP, Q19 BSS84, Q2 PSMN1R5-25MLHX, Q3 PSMN1R5-25MLHX, Q4 PSMN1R5-25MLHX, Q5 PSMN1R5-25MLHX, Q6 PSMN1R5-25MLHX, Q7 PSMN1R5-25MLHX, Q8 PSMN1R5-25MLHX, Q9 Si7141DP, U1 ADC104S021, U10 LTC2066IS5#TRPBF, U2 TMP390-Q1, U3 SN74LVC1G08DCK3, U4 TMP390-Q1, U5 MAX20096ATJ_VY+, U6 LTC4002ES8-8.4, U7 LTC2066IS5#TRPBF, U8 MAX17643, U9 MAX17643

Commit message: Merge revision 2.1 into main
Parts:
- added C65: 10uF, Capacitor_SMD:C_0805_2012Metric, F.Cu at (180.2, 131.2)
- added R56: 51k, Resistor_SMD:R_0805_2012Metric, F.Cu at (176.2, 131.2)
- added U11: 74AHC1G00, Package_TO_SOT_SMD:SOT-23-5, F.Cu at (187.0, 133.8)
- C58: value .1uF -> 10uF
- D16, D19, D3: footprint LED_SMD:LED_0805_2012Metric_Castellated -> LED_SMD:LED_0805_2012Metric
- moved C45 0.50 mm to (206.2, 119.5)
- moved C47 0.50 mm to (206.2, 124.5)
Connections:
- C59 pad 1: LASER_MON -> Net-(C59-Pad1)
- H1 pad 1: Net-(H1-Pad1) -> unconnected-(H1-Pad1)_1
- H2 pad 1: Net-(H2-Pad1) -> unconnected-(H2-Pad1)_2
- H3 pad 1: Net-(H3-Pad1) -> unconnected-(H3-Pad1)_3
- H4 pad 1: Net-(H4-Pad1) -> unconnected-(H4-Pad1)_6
- MCU1 pad 10: /TEC_ENABLE -> unconnected-(MCU1-Pin_10-Pad10)
- MCU1 pad 8: /CS_TEC_SET -> unconnected-(MCU1-Pin_8-Pad8)
- MCU1 pad 9: /CS_TEC_READ -> unconnected-(MCU1-Pin_9-Pad9)
- R54 pad 1: LASER_MON -> Net-(C59-Pad1)
- U10 pad 1: LASER_MON -> Net-(C59-Pad1)
- U2 pad 4: Net-(U2-Pad4) -> unconnected-(U2-~{OUTB}-Pad4)
- U4 pad 4: Net-(U4-Pad4) -> unconnected-(U4-~{OUTB}-Pad4)
- U5 pad 15: Net-(U5-Pad15) -> unconnected-(U5-IOUTV2-Pad15)
- U5 pad 26: Net-(U5-Pad26) -> unconnected-(U5-IOUTV1-Pad26)
- U8 pad 2: VDC -> Net-(U8-EN/UVLO)
- U8 pad 3: Net-(U8-Pad3) -> unconnected-(U8-~{RESET}-Pad3)
- U9 pad 3: Net-(U9-Pad3) -> unconnected-(U9-~{RESET}-Pad3)
- U9 pad 9: Net-(U9-Pad9) -> unconnected-(U9-EXTVCC-Pad9)
Routing:
- net ~{INTERLOCK_EN}: track 11.5 -> 146.0 mm, vias 0 -> 4
- net ~{CHARGE}: track 71.3 -> 144.0 mm, vias 2 -> 3
- net Net-(U8-EN/UVLO): track 0.00 -> 36.3 mm
- net Net-(C59-Pad1): track 0.00 -> 13.3 mm
- net LASER_MON: track 132.4 -> 125.3 mm
- net Net-(U7-+): track 17.2 -> 15.5 mm
- net +3V3: track 301.6 -> 303.2 mm, vias 29 -> 30
- net /LaserDriver/OUT2: track 76.7 -> 75.7 mm
- net Net-(R43-Pad2): track 14.0 -> 13.2 mm
- net +BATT: track 52.9 -> 52.3 mm
- net GND: vias 455 -> 459
- net VDC: vias 242 -> 238
- net Net-(U5-CSP2): vias 17 -> 18
- net Net-(U5-CSP1): vias 17 -> 18
Other:
- board text added: "Power Board Revision 1.6 Brian Pepin 2025"
- board text removed: "Power Board Revision 1.5 Brian Pepin 2021"
